Commit message: Guess physical values for mass and dimensions of hardware to create placeholder urdf. GIGI spawns in Gazebo Harmonic and sits still. Mass and dimension values need to be updated later once real hardware comes in

File: src/gigi_description/urdf/gigi.urdf.xacro (robot description, xacro)
@@ -1,4 +1,5 @@
 <?xml version="1.0"?>
 <robot xmlns:xacro="http://www.ros.org/wiki/xacro" name="my_bot"> <!-- allows for use of xacro -->
+    <xacro:include filename="inertial_macros.xacro"/> <!-- pulling in the inertial macros file, so xacro can stitch them together-->
   <!-- dimensions of hardware, update once you get kit; function like global variables -->
   <xacro:property name="chassis_length" value="0.30"/>
@@ -23,4 +24,11 @@
       <material name="blue"/>
     </visual>
+     <collision>
+        <origin xyz="0.10 0 ${chassis_height/2}" rpy="0 0 0"/>
+        <geometry><box size="${chassis_length} ${chassis_width} ${chassis_height}"/></geometry>
+    </collision>
+    <xacro:inertial_box mass="1.0" x="${chassis_length}" y="${chassis_width}" z="${chassis_height}">
+        <origin xyz="0.10 0 ${chassis_height/2}" rpy="0 0 0"/>
+    </xacro:inertial_box>
   </link>
   <!-- link between base_footprint and base_joint -->
@@ -30,5 +38,5 @@
     <origin xyz="0 0 ${wheel_radius}" rpy="0 0 0"/>
   </joint>
-  <!-- creating a template for a wheel that can be re-used for left and right wheels-->
+  <!-- creating a macro template for a wheel that can be re-used for left and right wheels-->
   <xacro:macro name="wheel" params="side y_reflect">
     <link name="${side}_wheel">
@@ -39,4 +47,10 @@
         <material name="dark"/>
       </visual>
+    <collision>
+        <geometry><cylinder radius="${wheel_radius}" length="${wheel_width}"/></geometry>
+    </collision>
+    <xacro:inertial_cylinder mass="0.1" length="${wheel_width}" radius="${wheel_radius}">
+        <origin xyz="0 0 0" rpy="0 0 0"/>
+    </xacro:inertial_cylinder>
     </link>
     <joint name="${side}_wheel_joint" type="continuous">
@@ -58,4 +72,10 @@
       <material name="dark"/>
     </visual>
+    <collision>
+        <geometry><sphere radius="${caster_radius}"/></geometry>
+    </collision>
+    <xacro:inertial_sphere mass="0.05" radius="${caster_radius}">
+        <origin xyz="0 0 0" rpy="0 0 0"/>
+    </xacro:inertial_sphere>
   </link>
   <!--caster wheel joint-->
